File: kicad/esp32-client.kicad_sch (KiCad schematic)
At the start: 0 parts

Commit message: init
Parts:
- added U?: ESP32-C3-MINI-1, PCM_Espressif:ESP32-C3-MINI-1, symbol PCM_Espressif:ESP32-C3-MINI-1
Connections:
- new net: U?.1 (GND), U?.11 (GND), U?.14 (GND), U?.2 (GND), U?.36 (GND), U?.37 (GND), U?.38 (GND), U?.39 (GND), U?.40 (GND), U?.41 (GND), U?.42 (GND), U?.43 (GND), U?.44 (GND), U?.45 (GND), U?.46 (GND), U?.47 (GND), U?.48 (GND), U?.49 (GND), U?.50 (GND), U?.51 (GND), U?.52 (GND), U?.53 (GND)
Changed lines of the file:
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@@
 	(generator_version "9.0")
 	(paper "A4")
+	(symbol
+		(lib_id "PCM_Espressif:ESP32-C3-MINI-1")
+		(at 127 78.74 0)
+		(unit 1)
+		(exclude_from_sim no)
+		(in_bom yes)
+		(on_board yes)
+		(dnp no)
+		(fields_autoplaced yes)
+		(property "Reference" "U?"
+			(at 129.1433 48.26 0)
+			(effects
+				(font
+					(size 1.27 1.27)
+				)
+				(justify left)
+			)
+		)
+		(property "Value" "ESP32-C3-MINI-1"
+			(at 129.1433 50.8 0)
+			(effects
+				(font
+					(size 1.27 1.27)
+				)
+				(justify left)
+			)
+		)
+		(property "Footprint" "PCM_Espressif:ESP32-C3-MINI-1"
+			(at 127 114.3 0)
+			(effects
+				(font
+					(size 1.27 1.27)
+				)
+				(hide yes)
+			)
+		)
+		(property "Datasheet" "https://www.espressif.com/sites/default/files/documentation/esp32-c3-mini-1_datasheet_en.pdf"
+			(at 127 116.84 0)
+			(effects
+				(font
+					(size 1.27 1.27)
+				)
+				(hide yes)
+			)
+		)
+		(property "Description" "ESP32-C3-MINI-1 family is an ultra-low-power MCU-based SoC solution that supports 2.4 GHz Wi-Fi and Bluetooth®Low Energy (Bluetooth LE)."
+			(at 127 78.74 0)
+			(effects
+				(font
+					(size 1.27 1.27)
+				)
+				(hide yes)
+			)
+		)
+		(pin "15"
+		)
+		(pin "43"
+		)
+		(pin "6"
+		)
+		(pin "10"
+		)
+		(pin "32"
+		)
+		(pin "46"
+		)
+		(pin "50"
+		)
+		(pin "42"
+		)
+		(pin "39"
+		)
+		(pin "45"
+		)
+		(pin "19"
+		)
+		(pin "49"
+		)
+		(pin "17"
+		)
+		(pin "29"
+		)
+		(pin "14"
+		)
+		(pin "31"
+		)
+		(pin "44"
+		)
+		(pin "20"
+		)
+		(pin "52"
+		)
+		(pin "2"
+		)
+		(pin "21"
+		)
+		(pin "24"
+		)
+		(pin "5"
+		)
+		(pin "53"
+		)
+		(pin "51"
+		)
+		(pin "34"
+		)
+		(pin "48"
+		)
+		(pin "11"
+		)
+		(pin "36"
+		)
+		(pin "26"
+		)
+		(pin "30"
+		)
+		(pin "27"
+		)
+		(pin "16"
+		)
+		(pin "23"
+		)
+		(pin "37"
+		)
+		(pin "9"
+		)
+		(pin "7"
+		)
+		(pin "4"
+		)
+		(pin "13"
+		)
+		(pin "12"
+		)
+		(pin "28"
+		)
+		(pin "8"
+		)
+		(pin "18"
+		)
+		(pin "22"
+		)
+		(pin "38"
+		)
+		(pin "35"
+		)
+		(pin "3"
+		)
+		(pin "25"
+		)
+		(pin "40"
+		)
+		(pin "47"
+		)
+		(pin "33"
+		)
+		(pin "1"
+		)
+		(pin "41"
+		)
+		(instances
+			(project ""
+				(path "/4a001952-2620-48e5-963e-8cfcd99c6e64"
+					(reference "U?")
+					(unit 1)
+				)
+			)
+		)
+	)
 	(sheet_instances
 		(path "/"

Commit message: init
Other:
- added sheet motor_driver (motor_driver.kicad_sch)
Changed lines of the file:
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@@
+		)
+	)
+	(sheet
+		(at 193.04 31.75)
+		(size 45.72 25.4)
+		(exclude_from_sim no)
+		(in_bom yes)
+		(on_board yes)
+		(dnp no)
+		(fields_autoplaced yes)
+		(stroke
+			(width 0.1524)
+			(type solid)
+		)
+		(fill
+			(color 0 0 0 0.0000)
+		)
+		(property "Sheetname" "motor_driver"
+			(at 193.04 31.0384 0)
+			(effects
+				(font
+					(size 1.27 1.27)
+				)
+				(justify left bottom)
+			)
+		)
+		(property "Sheetfile" "motor_driver.kicad_sch"
+			(at 193.04 57.7346 0)
+			(effects
+				(font
+					(size 1.27 1.27)
+				)
+				(justify left top)
+			)
+		)
+		(instances
+			(project "esp32-client"
+				(path "/4a001952-2620-48e5-963e-8cfcd99c6e64"
+					(page "2")
+				)
+			)
 		)
 	)

Commit message: init
Parts:
- gave numbers to parts that had none: 1
Changed lines of the file:
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@@
 		(dnp no)
 		(fields_autoplaced yes)
-		(property "Reference" "U?"
+		(property "Reference" "U1"
 			(at 129.1433 48.26 0)
 			(effects
@@
 			(project ""
 				(path "/4a001952-2620-48e5-963e-8cfcd99c6e64"
-					(reference "U?")
+					(reference "U1")
 					(unit 1)
 				)

Commit message: init
Connections:
- net GND: now reaches U1.1 (GND), U1.11 (GND), U1.14 (GND), U1.2 (GND), U1.36 (GND), U1.37 (GND), U1.38 (GND), U1.39 (GND), U1.40 (GND), U1.41 (GND), U1.42 (GND), U1.43 (GND), U1.44 (GND), U1.45 (GND), U1.46 (GND), U1.47 (GND), U1.48 (GND), U1.49 (GND), U1.50 (GND), U1.51 (GND), U1.52 (GND), U1.53 (GND)
- net +3.3V: now reaches U1.3 (3V3)
Other:
- added sheet power (power.kicad_sch)
Changed lines of the file:
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@@
 	(generator_version "9.0")
 	(paper "A4")
+	(wire
+		(pts
+			(xy 127 45.72) (xy 127 50.8)
+		)
+		(stroke
+			(width 0)
+			(type default)
+		)
+	)
+	(wire
+		(pts
+			(xy 127 106.68) (xy 127 109.22)
+		)
+		(stroke
+			(width 0)
+			(type default)
+		)
+	)
+	(symbol
+		(lib_id "power:+3.3V")
+		(at 127 45.72 0)
+		(unit 1)
+		(exclude_from_sim no)
+		(in_bom yes)
+		(on_board yes)
+		(dnp no)
+		(fields_autoplaced yes)
+		(property "Reference" "#PWR06"
+			(at 127 49.53 0)
+			(effects
+				(font
+					(size 1.27 1.27)
+				)
+				(hide yes)
+			)
+		)
+		(property "Value" "+3.3V"
+			(at 127 40.64 0)
+			(effects
+				(font
+					(size 1.27 1.27)
+				)
+			)
+		)
+		(property "Footprint" ""
+			(at 127 45.72 0)
+			(effects
+				(font
+					(size 1.27 1.27)
+				)
+				(hide yes)
+			)
+		)
+		(property "Datasheet" ""
+			(at 127 45.72 0)
+			(effects
+				(font
+					(size 1.27 1.27)
+				)
+				(hide yes)
+			)
+		)
+		(property "Description" "Power symbol creates a global label with name \"+3.3V\""
+			(at 127 45.72 0)
+			(effects
+				(font
+					(size 1.27 1.27)
+				)
+				(hide yes)
+			)
+		)
+		(pin "1"
+		)
+		(instances
+			(project ""
+				(path "/4a001952-2620-48e5-963e-8cfcd99c6e64"
+					(reference "#PWR06")
+					(unit 1)
+				)
+			)
+		)
+	)
 	(symbol
 		(lib_id "PCM_Espressif:ESP32-C3-MINI-1")
@@
 				)
 			)
+		)
+	)
+	(symbol
+		(lib_id "power:GND")
+		(at 127 109.22 0)
+		(unit 1)
+		(exclude_from_sim no)
+		(in_bom yes)
+		(on_board yes)
+		(dnp no)
+		(fields_autoplaced yes)
+		(property "Reference" "#PWR07"
+			(at 127 115.57 0)
+			(effects
+				(font
+					(size 1.27 1.27)
+				)
+				(hide yes)
+			)
+		)
+		(property "Value" "GND"
+			(at 127 114.3 0)
+			(effects
+				(font
+					(size 1.27 1.27)
+				)
+			)
+		)
+		(property "Footprint" ""
+			(at 127 109.22 0)
+			(effects
+				(font
+					(size 1.27 1.27)
+				)
+				(hide yes)
+			)
+		)
+		(property "Datasheet" ""
+			(at 127 109.22 0)
+			(effects
+				(font
+					(size 1.27 1.27)
+				)
+				(hide yes)
+			)
+		)
+		(property "Description" "Power symbol creates a global label with name \"GND\" , ground"
+			(at 127 109.22 0)
+			(effects
+				(font
+					(size 1.27 1.27)
+				)
+				(hide yes)
+			)
+		)
+		(pin "1"
+		)
+		(instances
+			(project ""
+				(path "/4a001952-2620-48e5-963e-8cfcd99c6e64"
+					(reference "#PWR07")
+					(unit 1)
+				)
+			)
+		)
+	)
+	(sheet
+		(at 40.64 137.16)
+		(size 35.56 25.4)
+		(exclude_from_sim no)
+		(in_bom yes)
+		(on_board yes)
+		(dnp no)
+		(fields_autoplaced yes)
+		(stroke
+			(width 0.1524)
+			(type solid)
+		)
+		(fill
+			(color 0 0 0 0.0000)
+		)
+		(property "Sheetname" "power"
+			(at 40.64 136.4484 0)
+			(effects
+				(font
+					(size 1.27 1.27)
+				)
+				(justify left bottom)
+			)
+		)
+		(property "Sheetfile" "power.kicad_sch"
+			(at 40.64 163.1446 0)
+			(effects
+				(font
+					(size 1.27 1.27)
+				)
+				(justify left top)
+			)
+		)
+		(instances
+			(project "esp32-client"
+				(path "/4a001952-2620-48e5-963e-8cfcd99c6e64"
+					(page "3")
+				)
+			)

Commit message: init
Parts:
- added C1: 100nF, symbol Device:C
- added R1: 10K, symbol Device:R
Connections:
- net +3.3V: now also R1.1
- net power/TXD: now reaches U1.30 (GPIO20/U0RXD)
- net power/RXD: now reaches U1.31 (GPIO21/U0TXD)
- net at U1.8 (EN/CHIP_PU): now also C1.1, R1.2
- new net power/RTS: C1.2
Other:
- sheet power ports: added RTS, RXD, TXD; removed none
- moved on the sheet: U1

Commit message: init
Parts:
- C1: value 100nF -> 1µF; footprint (none) -> Capacitor_SMD:C_1206_3216Metric
- R1: footprint (none) -> Resistor_SMD:R_0805_2012Metric
Connections:
- net power/RTS is gone; now on net GND: C1.2
- net +3.3V: now also R1.2; no longer R1.1
- net power/EN: now reaches C1.1, U1.8 (EN/CHIP_PU)
- net power/EN: now also R1.1; no longer R1.2
- net power/IO0: now reaches U1.12 (GPIO0/ADC1_CH0/XTAL_32K_P)
- net motor_driver/MOTOR_IN_1: now reaches U1.18 (GPIO4/ADC1_CH4)
- net motor_driver/MOTOR_IN_2: now reaches U1.19 (GPIO5/ADC2_CH0)
- net motor_driver/SLEEP: now reaches U1.20 (GPIO6)
- net motor_driver/MOTOR_OUT_1: now reaches U1.5 (GPIO2/ADC1_CH2)
- net motor_driver/MOTOR_OUT_2: now reaches U1.6 (GPIO3/ADC1_CH3)
- no-connect marks 0 -> 7
Other:
- sheet motor_driver ports: added MOTOR_IN_1, MOTOR_IN_2, MOTOR_OUT_1, MOTOR_OUT_2, SLEEP; removed none
- sheet power ports: added EN, IO0; removed RTS
- moved on the sheet: U1

Commit message: init
Parts:
- added H1, H2: MountingHole_Pad, MountingHole:MountingHole_2.5mm, symbol Mechanical:MountingHole_Pad
Connections:
- net GND: now also H1.1, H2.1
- net motor_driver/MOTOR_IN_1 renamed motor_driver/BIN_1_PWM
- net motor_driver/MOTOR_IN_2 renamed motor_driver/BIN_2_DIR
- net motor_driver/MOTOR_OUT_1 renamed motor_driver/AN_1_PWM
- net motor_driver/MOTOR_OUT_2 renamed motor_driver/AN_2_DIR
Other:
- sheet motor_driver ports: added AN_1_PWM, AN_2_DIR, BIN_1_PWM, BIN_2_DIR; removed MOTOR_IN_1, MOTOR_IN_2, MOTOR_OUT_1, MOTOR_OUT_2

Commit message: init
Parts:
- R1: footprint Resistor_SMD:R_0805_2012Metric -> Resistor_SMD:R_1206_3216Metric
Changed lines of the file:
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@@
 			)
 		)
-		(property "Footprint" "Resistor_SMD:R_0805_2012Metric"
+		(property "Footprint" "Resistor_SMD:R_1206_3216Metric"
 			(at 90.17 48.768 90)
 			(effects
