File: kicad/esp32-client.kicad_sch (KiCad schematic)
At the start: 5 parts, among them U1 ESP32-C3-MINI-1

Commit message: init
Connections:
- net power/D-: now reaches U1.26 (GPIO18/USB_D-)
- net power/D+: now reaches U1.27 (GPIO19/USB_D+)
- net power/EN: no longer names the net of C1.1, R1.1, U1.8 (EN/CHIP_PU)
- net power/IO0: no longer names the net of U1.12 (GPIO0/ADC1_CH0/XTAL_32K_P)
- net power/RXD: no longer names the net of U1.31 (GPIO21/U0TXD)
- net power/TXD: no longer names the net of U1.30 (GPIO20/U0RXD)
- no-connect marks 7 -> 8
Other:
- sheet power ports: added D+, D-; removed EN, IO0, RXD, TXD
Changed lines of the file:
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@@
-	)
-	(no_connect
-		(at 153.67 69.85)
 	)
 	(no_connect
@@
 	)
 	(no_connect
+		(at 97.79 59.69)
+	)
+	(no_connect
 		(at 153.67 92.71)
 	)
@@
 	)
 	(no_connect
-		(at 153.67 67.31)
-	)
-	(wire
-		(pts
-			(xy 82.55 54.61) (xy 82.55 125.73)
-		)
-		(stroke
-			(width 0)
-			(type default)
-		)
+		(at 153.67 62.23)
+	)
+	(no_connect
+		(at 153.67 59.69)
 	)
 	(wire
@@
 	(wire
 		(pts
-			(xy 78.74 59.69) (xy 78.74 125.73)
+			(xy 153.67 67.31) (xy 162.56 67.31)
 		)
 		(stroke
@@
 	(wire
 		(pts
-			(xy 153.67 59.69) (xy 167.64 59.69)
-		)
-		(stroke
-			(width 0)
-			(type default)
-		)
-	)
-	(wire
-		(pts
 			(xy 179.07 92.71) (xy 179.07 82.55)
 		)
@@
 	(wire
 		(pts
+			(xy 162.56 132.08) (xy 104.14 132.08)
+		)
+		(stroke
+			(width 0)
+			(type default)
+		)
+	)
+	(wire
+		(pts
 			(xy 93.98 46.99) (xy 125.73 46.99)
 		)
@@
 	(wire
 		(pts
+			(xy 162.56 67.31) (xy 162.56 132.08)
+		)
+		(stroke
+			(width 0)
+			(type default)
+		)
+	)
+	(wire
+		(pts
 			(xy 171.45 87.63) (xy 153.67 87.63)
 		)
@@
 	(wire
 		(pts
-			(xy 91.44 125.73) (xy 91.44 118.11)
-		)
-		(stroke
-			(width 0)
-			(type default)
-		)
-	)
-	(wire
-		(pts
 			(xy 76.2 54.61) (xy 82.55 54.61)
 		)
@@
 	(wire
 		(pts
+			(xy 165.1 69.85) (xy 165.1 135.89)
+		)
+		(stroke
+			(width 0)
+			(type default)
+		)
+	)
+	(wire
+		(pts
 			(xy 176.53 96.52) (xy 176.53 85.09)
 		)
@@
 	(wire
 		(pts
-			(xy 173.99 62.23) (xy 153.67 62.23)
-		)
-		(stroke
-			(width 0)
-			(type default)
-		)
-	)
-	(wire
-		(pts
-			(xy 167.64 118.11) (xy 167.64 59.69)
-		)
-		(stroke
-			(width 0)
-			(type default)
-		)
-	)
-	(wire
-		(pts
 			(xy 68.58 54.61) (xy 60.96 54.61)
 		)
@@
 	(wire
 		(pts
-			(xy 97.79 59.69) (xy 78.74 59.69)
-		)
-		(stroke
-			(width 0)
-			(type default)
-		)
-	)
-	(wire
-		(pts
 			(xy 179.07 82.55) (xy 153.67 82.55)
 		)
@@
 	(wire
 		(pts
+			(xy 165.1 135.89) (xy 104.14 135.89)
+		)
+		(stroke
+			(width 0)
+			(type default)
+		)
+	)
+	(wire
+		(pts
 			(xy 158.75 105.41) (xy 158.75 90.17)
 		)
@@
 	(wire
 		(pts
-			(xy 173.99 120.65) (xy 173.99 62.23)
-		)
-		(stroke
-			(width 0)
-			(type default)
-		)
-	)
-	(wire
-		(pts
 			(xy 193.04 100.33) (xy 171.45 100.33)
 		)
@@
 	(wire
 		(pts
+			(xy 153.67 69.85) (xy 165.1 69.85)
+		)
+		(stroke
+			(width 0)
+			(type default)
+		)
+	)
+	(wire
+		(pts
 			(xy 181.61 80.01) (xy 153.67 80.01)
 		)
@@
 		(pts
 			(xy 40.64 173.99) (xy 55.88 173.99)
-		)
-		(stroke
-			(width 0)
-			(type default)
-		)
-	)
-	(wire
-		(pts
-			(xy 95.25 125.73) (xy 95.25 120.65)
-		)
-		(stroke
-			(width 0)
-			(type default)
-		)
-	)
-	(wire
-		(pts
-			(xy 91.44 118.11) (xy 167.64 118.11)
-		)
-		(stroke
-			(width 0)
-			(type default)
-		)
-	)
-	(wire
-		(pts
-			(xy 95.25 120.65) (xy 173.99 120.65)
 		)
 		(stroke
@@
 			)
 		)
-		(pin "RXD" input
-			(at 91.44 125.73 90)
+		(pin "D+" input
+			(at 104.14 132.08 0)
 			(effects
 				(font
@@
 			)
 		)
-		(pin "TXD" input
-			(at 95.25 125.73 90)
-			(effects
-				(font
-					(size 1.27 1.27)
-				)
-				(justify right)
-			)
-		)
-		(pin "EN" input
-			(at 82.55 125.73 90)
-			(effects
-				(font
-					(size 1.27 1.27)
-				)
-				(justify right)
-			)
-		)
-		(pin "IO0" input
-			(at 78.74 125.73 90)
-			(effects
-				(font
+		(pin "D-" input
+			(at 104.14 135.89 0)
+			(effects
+				(font
