File: kicad/power.kicad_sch (KiCad schematic)
At the start: 12 parts, among them P1 USB_C_Plug_USB2.0, Q1 BCW66G, Q2 BCW66G, U2 USBLC6-2P6, U3 AMS1117-3.3

Commit message: init
Parts:
- removed Q1, Q2: BCW66G, Package_TO_SOT_SMD:SOT-23, symbol Simulation_SPICE:NPN
- removed R6, R7: 10K, Resistor_SMD:R_1206_3216Metric, symbol Device:R
- added C5: 100nF, Capacitor_SMD:C_1206_3216Metric, symbol Device:C
- added C6: 100nF, symbol Device:C
- gave numbers to parts that had none: 1
- renumbered C5 to C7, C7 to C8, D3 to D1, R10 to R3, U2 to U3, U3 to U5
Connections:
- net +3.3V: now also C6.1
- net +5V: now also C5.2
- net GND: now also C5.1, C6.2
- net RTS: now reaches U4.4 (~{RTS})
- net TXD: now reaches U4.8 (TXD)
- net RXD: now reaches U4.9 (RXD)
- no-connect marks 3 -> 4
Other:
- moved on the sheet: C7, C8, D1, R3, U5

Commit message: init
Parts:
- removed U4: CH340E, Package_SO:MSOP-10_3x3mm_P0.5mm, symbol Interface_USB:CH340E
- added U?: CH340C, Package_SO:SOIC-16_3.9x9.9mm_P1.27mm, symbol Interface_USB:CH340C
Connections:
- net +3.3V: now also U?.4 (V3)
- net +5V: now also U?.16 (VCC)
- net GND: now also U?.1 (GND)
- net RTS: now also U?.14 (~{RTS})
- net RXD: now also U?.3 (RXD)
- net TXD: now also U?.2 (TXD)
- net at U3.6 (I/O1): now also U?.5 (UD+)
- net at U3.4 (I/O2): now also U?.6 (UD-)
Changed lines of the file:
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@@
 	)
 	(symbol
-		(lib_id "Interface_USB:CH340E")
+		(lib_id "Interface_USB:CH340C")
 		(at 120.65 107.95 0)
 		(unit 1)
@@
 		(dnp no)
 		(fields_autoplaced yes)
-		(property "Reference" "U4"
+		(property "Reference" "U?"
 			(at 122.7933 123.19 0)
 			(effects
@@
 			)
 		)
-		(property "Value" "CH340E"
+		(property "Value" "CH340C"
 			(at 122.7933 125.73 0)
 			(effects
@@
 			)
 		)
-		(property "Footprint" "Package_SO:MSOP-10_3x3mm_P0.5mm"
-			(at 121.92 121.92 0)
+		(property "Footprint" "Package_SO:SOIC-16_3.9x9.9mm_P1.27mm"
+			(at 102.108 77.724 0)
 			(effects
 				(font
@@
 			)
 		)
-		(property "Datasheet" "https://www.mpja.com/download/35227cpdata.pdf"
-			(at 111.76 87.63 0)
+		(property "Datasheet" "https://datasheet.lcsc.com/szlcsc/Jiangsu-Qin-Heng-CH340C_C84681.pdf"
+			(at 114.046 74.676 0)
 			(effects
 				(font
@@
 			)
 		)
-		(property "Description" "USB serial converter, UART, MSOP-10"
-			(at 120.65 107.95 0)
+		(property "Description" "USB serial converter, crystal-less, UART, SOIC-16"
+			(at 119.126 71.882 0)
 			(effects
 				(font
@@
 			)
 		)
-		(pin "5"
+		(pin "1"
+		)
+		(pin "6"
+		)
+		(pin "14"
+		)
+		(pin "13"
+		)
+		(pin "12"
 		)
 		(pin "4"
 		)
+		(pin "5"
+		)
 		(pin "8"
+		)
+		(pin "16"
+		)
+		(pin "11"
 		)
 		(pin "2"
 		)
-		(pin "1"
+		(pin "10"
 		)
 		(pin "3"
-		)
-		(pin "10"
-		)
-		(pin "6"
 		)
 		(pin "7"
@@
 		(pin "9"
 		)
+		(pin "15"
+		)
 		(instances
 			(project ""
 				(path "/4a001952-2620-48e5-963e-8cfcd99c6e64/2cbfe13a-317f-4d7e-9177-61c47456d51b"
-					(reference "U4")
+					(reference "U?")
 					(unit 1)
 				)

Commit message: init
Parts:
- removed U?: CH340C, Package_SO:SOIC-16_3.9x9.9mm_P1.27mm, symbol Interface_USB:CH340C
- added C5: 10µF, Capacitor_SMD:C_1206_3216Metric, symbol Device:C
- added C7: 100pF, Capacitor_SMD:C_1206_3216Metric, symbol Device:C
- added C9: 100nF, Capacitor_SMD:C_1206_3216Metric, symbol Device:C
- added D1: GREEN, Diode_SMD:D_0603_1608Metric, symbol Device:LED
- added D2: RED, Diode_SMD:D_0603_1608Metric, symbol Device:LED
- added J1, J2: Conn_01x01_Pin, Connector_Pin:Pin_D1.3mm_L11.0mm, symbol Connector:Conn_01x01_Pin
- added Q1, Q2: BCW66G, Package_TO_SOT_SMD:SOT-23, symbol Simulation_SPICE:NPN
- added R10, R11: 10K, Resistor_SMD:R_0805_2012Metric, symbol Device:R
- added R3, R4, R8: 1K, Resistor_SMD:R_0805_2012Metric, symbol Device:R
- added R5: 1.2K, Resistor_SMD:R_0805_2012Metric, symbol Device:R
- added R6, R7: R, Resistor_SMD:R_0805_2012Metric, symbol Device:R
- added R9: 100, Resistor_SMD:R_0805_2012Metric, symbol Device:R
- added U3: TP4056-42-ESOP8, Package_SO:SOIC-8-1EP_3.9x4.9mm_P1.27mm_EP2.41x3.3mm_ThermalVias, symbol Battery_Management:TP4056-42-ESOP8
- added U4: U8205A, Package_TO_SOT_SMD:SOT-23-6, symbol PCM_yvolodym:8205A
- added U5: DW01A, Package_TO_SOT_SMD:SOT-23-6, symbol Battery_Management:DW01A
- added U7: CH340C, Package_SO:SOIC-16_3.9x9.9mm_P1.27mm, symbol Interface_USB:CH340C
- C6: value 100nF -> 10µF; footprint (none) -> Capacitor_SMD:C_1206_3216Metric
- R12: renamed from R3; footprint Resistor_SMD:R_1206_3216Metric -> Resistor_SMD:R_0805_2012Metric
- renumbered C7 to C10, C8 to C11, C5 to C8, D1 to D3, U3 to U6, U5 to U8
Connections:
- net +3.3V: no longer C6.1
- net +5V: now also C5.1, D1.2 (A), D2.2 (A), R6.2, U3.4 (V_{CC}), U3.8 (CE), U7.16 (VCC)
- net GND: now also C5.2, C9.2, J1.1 (Pin_1), R5.1, R7.1, R8.1, U3.3 (GND), U4.1 (S1), U4.3 (S2), U7.1 (GND)
- net RXD: now also U7.3 (RXD)
- net TXD: now also U7.2 (TXD)
- net at U6.6 (I/O1): now also U7.5 (UD+)
- net at U6.4 (I/O2): now also U7.6 (UD-)
- new net: D2.1 (K), R4.2
- new net: C9.1, U7.4 (V3)
- new net: C7.1, U5.6 (GND)
- new net: C7.2, R9.1, U5.5 (VCC)
- new net: R5.2, U3.2 (PROG)
- new net: R6.1, R7.2, U3.1 (TEMP)
- new net: C6.1, J2.1 (Pin_1), R9.2, U3.5 (BAT)
- new net: R8.2, U5.2 (CS)
- new net: D1.1 (K), R3.2
- new net: U4.4 (G2), U5.1 (OD)
- new net: U4.6 (G1), U5.3 (OC)
- new net: Q2.2 (B), R11.2
- new net: Q2.3 (E), R10.1, U7.13 (~{DTR})
- new net: R3.1, U3.6 (~{STDBY})
- new net: Q1.2 (B), R10.2
- new net: Q1.3 (E), R11.1, U7.14 (~{RTS})
- new net: R4.1, U3.7 (~{CHRG})
- new net EN: Q1.1 (C)
- new net IO0: Q2.1 (C)
- no-connect marks 4 -> 10
Other:
- note added: "Charger"
- moved on the sheet: C10, C11, C8, D3, P1, R12, U6, U8

Commit message: init
Parts:
- removed J1, J2: Conn_01x01_Pin, Connector_Pin:Pin_D1.3mm_L11.0mm, symbol Connector:Conn_01x01_Pin
- added J3: Conn_01x02, Connector_JST:JST_PH_B2B-PH-K_1x02_P2.00mm_Vertical, symbol Connector_Generic:Conn_01x02
Connections:
- net GND: now also U3.9 (EPAD), J3.2 (Pin_2)
- net at C6.1, R9.2, U3.5 (BAT): now also J3.1 (Pin_1)
- no-connect marks 10 -> 9

Commit message: init
Parts:
- R10, R11, R12, R3, R4, R5, R6, R7, R8, R9: footprint Resistor_SMD:R_0805_2012Metric -> Resistor_SMD:R_1206_3216Metric
Changed lines of the file:
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@@
 			)
 		)
-		(property "Footprint" "Resistor_SMD:R_0805_2012Metric"
+		(property "Footprint" "Resistor_SMD:R_1206_3216Metric"
 			(at 85.598 163.83 90)
 			(effects
@@
 			)
 		)
-		(property "Footprint" "Resistor_SMD:R_0805_2012Metric"
+		(property "Footprint" "Resistor_SMD:R_1206_3216Metric"
 			(at 105.918 162.56 90)
 			(effects
@@
 			)
 		)
-		(property "Footprint" "Resistor_SMD:R_0805_2012Metric"
+		(property "Footprint" "Resistor_SMD:R_1206_3216Metric"
 			(at 150.368 130.81 90)
 			(effects
@@
 			)
 		)
-		(property "Footprint" "Resistor_SMD:R_0805_2012Metric"
+		(property "Footprint" "Resistor_SMD:R_1206_3216Metric"
 			(at 114.808 154.94 90)
 			(effects
@@
 			)
 		)
-		(property "Footprint" "Resistor_SMD:R_0805_2012Metric"
+		(property "Footprint" "Resistor_SMD:R_1206_3216Metric"
 			(at 105.918 139.7 90)
 			(effects
@@
 			)
 		)
-		(property "Footprint" "Resistor_SMD:R_0805_2012Metric"
+		(property "Footprint" "Resistor_SMD:R_1206_3216Metric"
 			(at 32.258 147.32 90)
 			(effects
@@
 			)
 		)
-		(property "Footprint" "Resistor_SMD:R_0805_2012Metric"
+		(property "Footprint" "Resistor_SMD:R_1206_3216Metric"
 			(at 222.25 79.248 90)
 			(effects
@@
 			)
 		)
-		(property "Footprint" "Resistor_SMD:R_0805_2012Metric"
+		(property "Footprint" "Resistor_SMD:R_1206_3216Metric"
 			(at 221.742 35.56 90)
 			(effects
@@
 			)
 		)
-		(property "Footprint" "Resistor_SMD:R_0805_2012Metric"
+		(property "Footprint" "Resistor_SMD:R_1206_3216Metric"
 			(at 222.25 100.838 90)
 			(effects
@@
 			)
 		)
-		(property "Footprint" "Resistor_SMD:R_0805_2012Metric"
+		(property "Footprint" "Resistor_SMD:R_1206_3216Metric"
 			(at 47.498 147.32 90)
 			(effects

Commit message: init
Parts:
- removed C9: 100nF, Capacitor_SMD:C_1206_3216Metric, symbol Device:C
- removed Q1, Q2: BCW66G, Package_TO_SOT_SMD:SOT-23, symbol Simulation_SPICE:NPN
- removed R10, R11: 10K, Resistor_SMD:R_1206_3216Metric, symbol Device:R
- removed U7: CH340C, Package_SO:SOIC-16_3.9x9.9mm_P1.27mm, symbol Interface_USB:CH340C
Connections:
- net +3.3V: now also C6.1, J3.1 (Pin_1), R9.1, U3.5 (BAT)
- net GND: no longer J3.2 (Pin_2), U4.3 (S2)
- net at C7.1, U5.6 (GND): now also J3.2 (Pin_2), U4.3 (S2)
- net at C7.2, U5.5 (VCC): now also R9.2; no longer R9.1
- net D+: now reaches U6.6 (I/O1)
- net D-: now reaches U6.4 (I/O2)
- no-connect marks 9 -> 4
Other:
- moved on the sheet: C10, C11, C7, C8, D3, P1, R12, R9, U6, U8

Commit message: init
Changed lines of the file:
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@@
 	(wire
 		(pts
+			(xy 95.25 130.81) (xy 148.59 130.81)
+		)
+		(stroke
+			(width 0)
+			(type default)
+		)
+	)
+	(wire
+		(pts
 			(xy 113.03 158.75) (xy 113.03 170.18)
 		)
@@
 	(wire
 		(pts
-			(xy 95.25 130.81) (xy 148.59 130.81)
-		)
-		(stroke
-			(width 0)
-			(type default)
-		)
-	)
-	(wire
-		(pts
 			(xy 113.03 146.05) (xy 113.03 151.13)
 		)
@@
 	(wire
 		(pts
+			(xy 146.05 137.16) (xy 146.05 140.97)
+		)
+		(stroke
+			(width 0)
+			(type default)
+		)
+	)
+	(wire
+		(pts
 			(xy 77.47 80.01) (xy 77.47 83.82)
 		)
@@
 	(wire
 		(pts
+			(xy 146.05 170.18) (xy 146.05 172.72)
+		)
+		(stroke
+			(width 0)
+			(type default)
+		)
+	)
+	(wire
+		(pts
 			(xy 30.48 124.46) (xy 30.48 127)
 		)
@@
 	)
 	(symbol
+		(lib_id "power:PWR_FLAG")
+		(at 146.05 172.72 180)
+		(unit 1)
+		(exclude_from_sim no)
+		(in_bom yes)
+		(on_board yes)
+		(dnp no)
+		(fields_autoplaced yes)
+		(property "Reference" "#FLG05"
+			(at 146.05 174.625 0)
+			(effects
+				(font
+					(size 1.27 1.27)
+				)
+				(hide yes)
+			)
+		)
+		(property "Value" "PWR_FLAG"
+			(at 146.05 177.8 0)
+			(effects
+				(font
+					(size 1.27 1.27)
+				)
+			)
+		)
+		(property "Footprint" ""
+			(at 146.05 172.72 0)
+			(effects
+				(font
+					(size 1.27 1.27)
+				)
+				(hide yes)
+			)
+		)
+		(property "Datasheet" "~"
+			(at 146.05 172.72 0)
+			(effects
+				(font
+					(size 1.27 1.27)
+				)
+				(hide yes)
+			)
+		)
+		(property "Description" "Special symbol for telling ERC where power comes from"
+			(at 146.05 172.72 0)
+			(effects
+				(font
+					(size 1.27 1.27)
+				)
+				(hide yes)
+			)
+		)
+		(pin "1"
+		)
+		(instances
+			(project ""
+				(path "/4a001952-2620-48e5-963e-8cfcd99c6e64/2cbfe13a-317f-4d7e-9177-61c47456d51b"
+					(reference "#FLG05")
+					(unit 1)
+				)
+			)
+		)
+	)
+	(symbol
 		(lib_id "power:+3.3V")
 		(at 148.59 125.73 0)
@@
 					(unit 1)
 				)
+			)
+		)
+	)
+	(symbol
+		(lib_id "power:PWR_FLAG")
+		(at 146.05 137.16 0)
+		(unit 1)
+		(exclude_from_sim no)
+		(in_bom yes)
+		(on_board yes)
+		(dnp no)
+		(property "Reference" "#FLG03"
+			(at 146.05 135.255 0)
+			(effects
+				(font
+					(size 1.27 1.27)
+				)
+				(hide yes)
+			)
+		)
+		(property "Value" "PWR_FLAG"
+			(at 142.748 133.35 0)
+			(effects
+				(font
+					(size 1.27 1.27)
+				)
+			)
+		)
+		(property "Footprint" ""
+			(at 146.05 137.16 0)
+			(effects
+				(font
+					(size 1.27 1.27)
+				)
+				(hide yes)
+			)
+		)
+		(property "Datasheet" "~"
+			(at 146.05 137.16 0)
+			(effects
+				(font
+					(size 1.27 1.27)
+				)
+				(hide yes)
+			)
+		)
+		(property "Description" "Special symbol for telling ERC where power comes from"
+			(at 146.05 137.16 0)
+			(effects
+				(font
+					(size 1.27 1.27)
+				)
+				(hide yes)
+			)
+		)
+		(pin "1"
+		)
+		(instances
+			(project ""
+				(path "/4a001952-2620-48e5-963e-8cfcd99c6e64/2cbfe13a-317f-4d7e-9177-61c47456d51b"
+					(reference "#FLG03")
+					(unit 1)
+				)
