File: kicad/power.kicad_sch (KiCad schematic)
At the start: 24 parts, among them J3 Conn_01x02, P1 USB_C_Plug_USB2.0, U3 TP4056-42-ESOP8, U4 U8205A, U5 DW01A, U6 USBLC6-2P6, U8 AMS1117-3.3

Commit message: init
Parts:
- added U7: ~, PCM_yvolodym:Switch, symbol PCM_yvolodym:Switch small
- renumbered C8 to C10, C10 to C8, C11 to C9, R9 to R10, R12 to R9, U6 to U4, U4 to U5, U5 to U6
Connections:
- net at C7.1, U5.3 (S2), U6.6 (GND): now also U7.3; no longer J3.2 (Pin_2)
- new net: J3.2 (Pin_2), U7.2
- no-connect marks 4 -> 5
Changed lines of the file:
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@@
 	)
 	(no_connect
+		(at 149.86 161.29)
+	)
+	(no_connect
 		(at 128.27 154.94)
 	)
@@
 	(wire
 		(pts
-			(xy 146.05 170.18) (xy 160.02 170.18)
+			(xy 113.03 170.18) (xy 104.14 170.18)
 		)
 		(stroke
@@
 	(wire
 		(pts
-			(xy 113.03 170.18) (xy 104.14 170.18)
+			(xy 139.7 39.37) (xy 139.7 43.18)
 		)
 		(stroke
@@
 	(wire
 		(pts
-			(xy 139.7 39.37) (xy 139.7 43.18)
+			(xy 54.61 127) (xy 45.72 127)
 		)
 		(stroke
@@
 	(wire
 		(pts
-			(xy 54.61 127) (xy 45.72 127)
+			(xy 160.02 161.29) (xy 160.02 149.86)
 		)
 		(stroke
@@
 	(wire
 		(pts
+			(xy 154.94 170.18) (xy 146.05 170.18)
+		)
+		(stroke
+			(width 0)
+			(type default)
+		)
+	)
+	(wire
+		(pts
 			(xy 140.97 146.05) (xy 140.97 170.18)
 		)
@@
 	(wire
 		(pts
+			(xy 154.94 167.64) (xy 154.94 170.18)
+		)
+		(stroke
+			(width 0)
+			(type default)
+		)
+	)
+	(wire
+		(pts
 			(xy 69.85 80.01) (xy 77.47 80.01)
 		)
@@
 	(wire
 		(pts
-			(xy 160.02 170.18) (xy 160.02 149.86)
-		)
-		(stroke
-			(width 0)
-			(type default)
-		)
-	)
-	(wire
-		(pts
 			(xy 83.82 157.48) (xy 83.82 160.02)
 		)
@@
 		(dnp no)
 		(fields_autoplaced yes)
-		(property "Reference" "#PWR023"
+		(property "Reference" "#PWR019"
 			(at 187.96 78.74 0)
 			(effects
@@
 			(project "esp32-client"
 				(path "/4a001952-2620-48e5-963e-8cfcd99c6e64/2cbfe13a-317f-4d7e-9177-61c47456d51b"
-					(reference "#PWR023")
+					(reference "#PWR019")
 					(unit 1)
 				)
@@
 		(dnp no)
 		(fields_autoplaced yes)
-		(property "Reference" "#PWR015"
+		(property "Reference" "#PWR014"
 			(at 106.68 59.69 0)
 			(effects
@@
 			(project "esp32-client"
 				(path "/4a001952-2620-48e5-963e-8cfcd99c6e64/2cbfe13a-317f-4d7e-9177-61c47456d51b"
-					(reference "#PWR015")
+					(reference "#PWR014")
 					(unit 1)
 				)
@@
 		(dnp no)
 		(fields_autoplaced yes)
-		(property "Reference" "#PWR019"
+		(property "Reference" "#PWR016"
 			(at 127 38.1 0)
 			(effects
@@
 			(project "esp32-client"
 				(path "/4a001952-2620-48e5-963e-8cfcd99c6e64/2cbfe13a-317f-4d7e-9177-61c47456d51b"
-					(reference "#PWR019")
+					(reference "#PWR016")
 					(unit 1)
 				)
@@
 		(dnp no)
 		(fields_autoplaced yes)
-		(property "Reference" "C10"
+		(property "Reference" "C8"
 			(at 153.67 45.7199 0)
 			(effects
@@
 			(project "esp32-client"
 				(path "/4a001952-2620-48e5-963e-8cfcd99c6e64/2cbfe13a-317f-4d7e-9177-61c47456d51b"
-					(reference "C10")
+					(reference "C8")
 					(unit 1)
 				)
@@
 		(dnp no)
 		(fields_autoplaced yes)
-		(property "Reference" "#PWR022"
+		(property "Reference" "#PWR018"
 			(at 187.96 40.64 0)
 			(effects
@@
 			(project "esp32-client"
 				(path "/4a001952-2620-48e5-963e-8cfcd99c6e64/2cbfe13a-317f-4d7e-9177-61c47456d51b"
-					(reference "#PWR022")
+					(reference "#PWR018")
 					(unit 1)
 				)
@@
 		(dnp no)
 		(fields_autoplaced yes)
-		(property "Reference" "R9"
+		(property "Reference" "R10"
 			(at 153.67 134.62 90)
 			(effects
@@
 			(project "esp32-client"
 				(path "/4a001952-2620-48e5-963e-8cfcd99c6e64/2cbfe13a-317f-4d7e-9177-61c47456d51b"
-					(reference "R9")
+					(reference "R10")
 					(unit 1)
 				)
@@
 		(dnp no)
 		(fields_autoplaced yes)
-		(property "Reference" "C8"
+		(property "Reference" "C10"
 			(at 212.09 124.4599 0)
 			(effects
@@
 			(project ""
 				(path "/4a001952-2620-48e5-963e-8cfcd99c6e64/2cbfe13a-317f-4d7e-9177-61c47456d51b"
-					(reference "C8")
+					(reference "C10")
+					(unit 1)
+				)
+			)
+		)
+	)
+	(symbol
+		(lib_id "PCM_yvolodym:Switch small")
+		(at 154.94 158.75 0)
+		(unit 1)
+		(exclude_from_sim no)
+		(in_bom yes)
+		(on_board yes)
+		(dnp no)
+		(fields_autoplaced yes)
+		(property "Reference" "U7"
+			(at 154.94 154.94 0)
+			(effects
+				(font
+					(size 1.27 1.27)
+				)
+			)
+		)
+		(property "Value" "~"
+			(at 154.94 157.48 0)
+			(effects
+				(font
+					(size 1.27 1.27)
+				)
+			)
+		)
+		(property "Footprint" "PCM_yvolodym:Switch"
+			(at 154.686 155.956 0)
+			(effects
+				(font
+					(size 1.27 1.27)
+				)
+				(hide yes)
+			)
+		)
+		(property "Datasheet" ""
+			(at 154.94 158.75 0)
+			(effects
+				(font
+					(size 1.27 1.27)
+				)
+				(hide yes)
+			)
+		)
+		(property "Description" ""
+			(at 154.94 158.75 0)
+			(effects
+				(font
+					(size 1.27 1.27)
+				)
+				(hide yes)
+			)
+		)
+		(pin "2"
+		)
+		(pin "3"
+		)
+		(pin "1"
+		)
+		(instances
+			(project ""
+				(path "/4a001952-2620-48e5-963e-8cfcd99c6e64/2cbfe13a-317f-4d7e-9177-61c47456d51b"
+					(reference "U7")
 					(unit 1)
 				)
@@
 		(dnp no)
 		(fields_autoplaced yes)
-		(property "Reference" "#PWR016"
+		(property "Reference" "#PWR015"
 			(at 116.84 43.18 0)
 			(effects
@@
 			(project "esp32-client"
 				(path "/4a001952-2620-48e5-963e-8cfcd99c6e64/2cbfe13a-317f-4d7e-9177-61c47456d51b"
-					(reference "#PWR016")
+					(reference "#PWR015")
 					(unit 1)
 				)
@@
 		(dnp no)
 		(fields_autoplaced yes)
-		(property "Reference" "C11"
+		(property "Reference" "C9"
 			(at 191.77 45.7199 0)
 			(effects
@@
 			(project "esp32-client"
 				(path "/4a001952-2620-48e5-963e-8cfcd99c6e64/2cbfe13a-317f-4d7e-9177-61c47456d51b"
-					(reference "C11")
+					(reference "C9")
 					(unit 1)
 				)
@@
 		(on_board yes)
 		(dnp no)
-		(property "Reference" "U5"
+		(property "Reference" "U6"
 			(at 127 133.35 0)
 			(effects
@@
 			(project "esp32-client"
 				(path "/4a001952-2620-48e5-963e-8cfcd99c6e64/2cbfe13a-317f-4d7e-9177-61c47456d51b"
-					(reference "U5")
+					(reference "U6")
 					(unit 1)
 				)
@@
 		(on_board yes)
 		(dnp no)
-		(property "Reference" "U4"
+		(property "Reference" "U5"
 			(at 118.11 162.052 90)
 			(effects
@@
 			(project "esp32-client"
 				(path "/4a001952-2620-48e5-963e-8cfcd99c6e64/2cbfe13a-317f-4d7e-9177-61c47456d51b"
-					(reference "U4")
+					(reference "U5")
 					(unit 1)
 				)
@@
 		(dnp no)
 		(fields_autoplaced yes)
-		(property "Reference" "#PWR018"
+		(property "Reference" "#PWR021"
 			(at 208.28 138.43 0)
 			(effects
@@
 			(project ""
 				(path "/4a001952-2620-48e5-963e-8cfcd99c6e64/2cbfe13a-317f-4d7e-9177-61c47456d51b"
-					(reference "#PWR018")
+					(reference "#PWR021")
 					(unit 1)
 				)
@@
 		(dnp no)
 		(fields_autoplaced yes)
-		(property "Reference" "R12"
+		(property "Reference" "R9"
 			(at 142.24 45.7199 0)
 			(effects
@@
 			(project "esp32-client"
 				(path "/4a001952-2620-48e5-963e-8cfcd99c6e64/2cbfe13a-317f-4d7e-9177-61c47456d51b"
-					(reference "R12")
+					(reference "R9")
 					(unit 1)
 				)
@@
 		(dnp no)
 		(fields_autoplaced yes)
-		(property "Reference" "#PWR020"
+		(property "Reference" "#PWR017"
 			(at 148.59 129.54 0)
 			(effects
@@
 			(project "esp32-client"
 				(path "/4a001952-2620-48e5-963e-8cfcd99c6e64/2cbfe13a-317f-4d7e-9177-61c47456d51b"
-					(reference "#PWR020")
+					(reference "#PWR017")
 					(unit 1)
 				)
@@
 		(dnp no)
 		(fields_autoplaced yes)
-		(property "Reference" "#FLG04"
+		(property "Reference" "#FLG03"
 			(at 114.3 32.385 0)
 			(effects
@@
 			(project "esp32-client"
 				(path "/4a001952-2620-48e5-963e-8cfcd99c6e64/2cbfe13a-317f-4d7e-9177-61c47456d51b"
-					(reference "#FLG04")
+					(reference "#FLG03")
 					(unit 1)
 				)
@@
 		(on_board yes)
 		(dnp no)
-		(property "Reference" "#FLG03"
+		(property "Reference" "#FLG04"
 			(at 146.05 135.255 0)
 			(effects
@@
 			(project ""
 				(path "/4a001952-2620-48e5-963e-8cfcd99c6e64/2cbfe13a-317f-4d7e-9177-61c47456d51b"
-					(reference "#FLG03")
+					(reference "#FLG04")
 					(unit 1)
 				)
@@
 		(on_board yes)
 		(dnp no)
-		(property "Reference" "U6"
+		(property "Reference" "U4"
 			(at 112.776 49.276 0)
 			(effects
@@
 			(project "esp32-client"
 				(path "/4a001952-2620-48e5-963e-8cfcd99c6e64/2cbfe13a-317f-4d7e-9177-61c47456d51b"
-					(reference "U6")
+					(reference "U4")
 					(unit 1)
 				)
@@
 		(dnp no)
 		(fields_autoplaced yes)
-		(property "Reference" "#PWR017"
+		(property "Reference" "#PWR020"
 			(at 208.28 124.46 0)
 			(effects
@@
 			(project ""
 				(path "/4a001952-2620-48e5-963e-8cfcd99c6e64/2cbfe13a-317f-4d7e-9177-61c47456d51b"
-					(reference "#PWR017")
+					(reference "#PWR020")
 					(unit 1)
 				)
