File: kicad/motor_driver.kicad_sch (KiCad schematic)
At the start: 1 part

Commit message: init
Parts:
- removed U?: DRV8833PW, Package_SO:TSSOP-16_4.4x5mm_P0.65mm, symbol Driver_Motor:DRV8833PW
- added C1: 10µF, Capacitor_THT:CP_Radial_D5.0mm_P2.00mm, symbol Device:C_Polarized
- added C2: 100pF, Capacitor_SMD:C_1206_3216Metric, symbol Device:C
- added C3: 2,2µF, Capacitor_SMD:C_1206_3216Metric, symbol Device:C
- added R1: 0,68Ω, Resistor_SMD:R_1206_3216Metric, symbol Device:R
- added U2: DRV8833PW, Package_SO:TSSOP-16_4.4x5mm_P0.65mm, symbol Driver_Motor:DRV8833PW
Connections:
- new net: R1.1, U2.3 (AISEN), U2.6 (BISEN)
- new net: C3.2, U2.14 (VINT)
- new net: C2.2, U2.11 (VCP)
- new net +3V3: C1.1, C2.1, U2.12 (VM)
- new net GND: C1.2, C3.1, R1.2, U2.13 (GND)
- new net MOTOR_IN_1: U2.16 (AIN1), U2.9 (BIN1)
- new net MOTOR_IN_2: U2.10 (BIN2), U2.15 (AIN2)
- new net MOTOR_OUT_1: U2.2 (AOUT1), U2.7 (BOUT1)
- new net MOTOR_OUT_2: U2.4 (AOUT2), U2.5 (BOUT2)
- new net SLEEP: U2.1 (~{SLEEP})
- no-connect marks 0 -> 1

Commit message: init
Connections:
- net +3V3 renamed +3.3V
Changed lines of the file:
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@@
+	)
+	(symbol
+		(lib_id "power:+3.3V")
+		(at 158.75 67.31 0)
+		(unit 1)
+		(exclude_from_sim no)
+		(in_bom yes)
+		(on_board yes)
+		(dnp no)
+		(fields_autoplaced yes)
+		(property "Reference" "#PWR05"
+			(at 158.75 71.12 0)
+			(effects
+				(font
+					(size 1.27 1.27)
+				)
+				(hide yes)
+			)
+		)
+		(property "Value" "+3.3V"
+			(at 158.75 62.23 0)
+			(effects
+				(font
+					(size 1.27 1.27)
+				)
+			)
+		)
+		(property "Footprint" ""
+			(at 158.75 67.31 0)
+			(effects
+				(font
+					(size 1.27 1.27)
+				)
+				(hide yes)
+			)
+		)
+		(property "Datasheet" ""
+			(at 158.75 67.31 0)
+			(effects
+				(font
+					(size 1.27 1.27)
+				)
+				(hide yes)
+			)
+		)
+		(property "Description" "Power symbol creates a global label with name \"+3.3V\""
+			(at 158.75 67.31 0)
+			(effects
+				(font
+					(size 1.27 1.27)
+				)
+				(hide yes)
+			)
+		)
+		(pin "1"
+		)
+		(instances
+			(project ""
+				(path "/4a001952-2620-48e5-963e-8cfcd99c6e64/53c57007-9e2c-4812-92db-21a9e5c7f42c"
+					(reference "#PWR05")
+					(unit 1)
+				)
+			)
+		)
 	)
 	(symbol
@@
 					(unit 1)
 				)
-			)
-		)
-	)
-	(symbol
-		(lib_id "power:+3V3")
-		(at 158.75 67.31 0)
-		(unit 1)
-		(exclude_from_sim no)
-		(in_bom yes)
-		(on_board yes)
-		(dnp no)
-		(fields_autoplaced yes)
-		(property "Reference" "#PWR05"
-			(at 158.75 71.12 0)
-			(effects
-				(font
-					(size 1.27 1.27)
-				)
-				(hide yes)
-			)
-		)
-		(property "Value" "+3V3"
-			(at 158.75 62.23 0)
-			(effects
-				(font
-					(size 1.27 1.27)
-				)
-			)
-		)
-		(property "Footprint" ""
-			(at 158.75 67.31 0)
-			(effects
-				(font
-					(size 1.27 1.27)
-				)
-				(hide yes)
-			)
-		)
-		(property "Datasheet" ""
-			(at 158.75 67.31 0)
-			(effects
-				(font
-					(size 1.27 1.27)
-				)
-				(hide yes)
-			)
-		)
-		(property "Description" "Power symbol creates a global label with name \"+3V3\""
-			(at 158.75 67.31 0)
-			(effects
-				(font
-					(size 1.27 1.27)
-				)
-				(hide yes)
-			)
-		)
-		(pin "1"
-		)
-		(instances
-			(project "esp32-client"
-				(path "/4a001952-2620-48e5-963e-8cfcd99c6e64/53c57007-9e2c-4812-92db-21a9e5c7f42c"
-					(reference "#PWR05")
-					(unit 1)
-				)

Commit message: init
Parts:
- renumbered C1 to C2, C2 to C3, C3 to C4, R1 to R2
Changed lines of the file:
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@@
 		(on_board yes)
 		(dnp no)
-		(property "Reference" "#PWR03"
+		(property "Reference" "#PWR06"
 			(at 134.62 82.55 0)
 			(effects
@@
 			(project "esp32-client"
 				(path "/4a001952-2620-48e5-963e-8cfcd99c6e64/53c57007-9e2c-4812-92db-21a9e5c7f42c"
-					(reference "#PWR03")
+					(reference "#PWR06")
 					(unit 1)
 				)
@@
 		(dnp no)
 		(fields_autoplaced yes)
-		(property "Reference" "#PWR01"
+		(property "Reference" "#PWR04"
 			(at 104.14 124.46 0)
 			(effects
@@
 			(project "esp32-client"
 				(path "/4a001952-2620-48e5-963e-8cfcd99c6e64/53c57007-9e2c-4812-92db-21a9e5c7f42c"
-					(reference "#PWR01")
+					(reference "#PWR04")
 					(unit 1)
 				)
@@
 		(on_board yes)
 		(dnp no)
-		(property "Reference" "R1"
+		(property "Reference" "R2"
 			(at 97.79 108.712 0)
 			(effects
@@
 			(project "esp32-client"
 				(path "/4a001952-2620-48e5-963e-8cfcd99c6e64/53c57007-9e2c-4812-92db-21a9e5c7f42c"
-					(reference "R1")
+					(reference "R2")
 					(unit 1)
 				)
@@
 		(on_board yes)
 		(dnp no)
-		(property "Reference" "C3"
+		(property "Reference" "C4"
 			(at 148.336 87.376 90)
 			(effects
@@
 			(project "esp32-client"
 				(path "/4a001952-2620-48e5-963e-8cfcd99c6e64/53c57007-9e2c-4812-92db-21a9e5c7f42c"
-					(reference "C3")
+					(reference "C4")
 					(unit 1)
 				)
@@
 		(dnp no)
 		(fields_autoplaced yes)
-		(property "Reference" "#PWR04"
+		(property "Reference" "#PWR07"
 			(at 151.13 127 0)
 			(effects
@@
 			(project "esp32-client"
 				(path "/4a001952-2620-48e5-963e-8cfcd99c6e64/53c57007-9e2c-4812-92db-21a9e5c7f42c"
-					(reference "#PWR04")
+					(reference "#PWR07")
 					(unit 1)
 				)
@@
 		(dnp no)
 		(fields_autoplaced yes)
-		(property "Reference" "#PWR05"
+		(property "Reference" "#PWR08"
 			(at 158.75 71.12 0)
 			(effects
@@
 			(project ""
 				(path "/4a001952-2620-48e5-963e-8cfcd99c6e64/53c57007-9e2c-4812-92db-21a9e5c7f42c"
-					(reference "#PWR05")
+					(reference "#PWR08")
 					(unit 1)
 				)
@@
 		(on_board yes)
 		(dnp no)
-		(property "Reference" "C1"
+		(property "Reference" "C2"
 			(at 105.156 80.518 0)
 			(effects
@@
 			(project "esp32-client"
 				(path "/4a001952-2620-48e5-963e-8cfcd99c6e64/53c57007-9e2c-4812-92db-21a9e5c7f42c"
-					(reference "C1")
+					(reference "C2")
 					(unit 1)
 				)
@@
 		(dnp no)
 		(fields_autoplaced yes)
-		(property "Reference" "C2"
+		(property "Reference" "C3"
 			(at 127 80.0099 0)
 			(effects
@@
 			(project "esp32-client"
 				(path "/4a001952-2620-48e5-963e-8cfcd99c6e64/53c57007-9e2c-4812-92db-21a9e5c7f42c"
-					(reference "C2")
+					(reference "C3")
 					(unit 1)
 				)
@@
 		(dnp no)
 		(fields_autoplaced yes)
-		(property "Reference" "#PWR02"
+		(property "Reference" "#PWR05"
 			(at 114.3 93.98 0)
 			(effects
@@
 			(project "esp32-client"
 				(path "/4a001952-2620-48e5-963e-8cfcd99c6e64/53c57007-9e2c-4812-92db-21a9e5c7f42c"
-					(reference "#PWR02")
-					(unit 1)
-				)
+					(reference "#PWR05")
+					(unit 1)
+				)

Commit message: init
Parts:
- R2: footprint Resistor_SMD:R_1206_3216Metric -> Resistor_SMD:R_0805_2012Metric
Changed lines of the file:
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@@
 			)
 		)
-		(property "Footprint" "Resistor_SMD:R_1206_3216Metric"
+		(property "Footprint" "Resistor_SMD:R_0805_2012Metric"
 			(at 102.362 110.49 90)
 			(effects

Commit message: init
Parts:
- added J1, J2: Conn_01x01_Pin, Connector_Pin:Pin_D1.0mm_L10.0mm, symbol Connector:Conn_01x01_Pin
Connections:
- net MOTOR_IN_1 renamed AN_1_PWM
- net AN_1_PWM: no longer U2.9 (BIN1)
- net MOTOR_IN_2 renamed AN_2_DIR
- net AN_2_DIR: no longer U2.10 (BIN2)
- net MOTOR_OUT_1: no longer names the net of U2.2 (AOUT1), U2.7 (BOUT1)
- net MOTOR_OUT_1: now also J1.1 (Pin_1)
- net MOTOR_OUT_2: no longer names the net of U2.4 (AOUT2), U2.5 (BOUT2)
- net MOTOR_OUT_2: now also J2.1 (Pin_1)
- new net BIN_1_PWM: U2.9 (BIN1)
- new net BIN_2_DIR: U2.10 (BIN2)
Changed lines of the file:
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@@
 	(paper "A4")
-	(junction
-		(at 133.35 105.41)
-		(diameter 0)
-		(color 0 0 0 0)
-	)
 	(junction
 		(at 158.75 72.39)
@@
 	)
 	(junction
-		(at 135.89 113.03)
-		(diameter 0)
-		(color 0 0 0 0)
-	)
-	(junction
 		(at 132.08 100.33)
 		(diameter 0)
@@
 	(wire
 		(pts
-			(xy 135.89 107.95) (xy 135.89 113.03)
-		)
-		(stroke
-			(width 0)
-			(type default)
-		)
-	)
-	(wire
-		(pts
 			(xy 156.21 87.63) (xy 156.21 82.55)
 		)
@@
 	(wire
 		(pts
-			(xy 138.43 107.95) (xy 135.89 107.95)
-		)
-		(stroke
-			(width 0)
-			(type default)
-		)
-	)
-	(wire
-		(pts
 			(xy 156.21 82.55) (xy 152.4 82.55)
 		)
@@
 	(wire
 		(pts
+			(xy 128.27 110.49) (xy 138.43 110.49)
+		)
+		(stroke
+			(width 0)
+			(type default)
+		)
+	)
+	(wire
+		(pts
 			(xy 173.99 110.49) (xy 173.99 105.41)
 		)
@@
 	(wire
 		(pts
-			(xy 135.89 113.03) (xy 138.43 113.03)
-		)
-		(stroke
-			(width 0)
-			(type default)
-		)
-	)
-	(wire
-		(pts
-			(xy 128.27 113.03) (xy 135.89 113.03)
-		)
-		(stroke
-			(width 0)
-			(type default)
-		)
-	)
-	(wire
-		(pts
 			(xy 140.97 82.55) (xy 144.78 82.55)
 		)
@@
 	(wire
 		(pts
-			(xy 138.43 110.49) (xy 133.35 110.49)
-		)
-		(stroke
-			(width 0)
-			(type default)
-		)
-	)
-	(wire
-		(pts
 			(xy 163.83 105.41) (xy 173.99 105.41)
 		)
@@
 	(wire
 		(pts
-			(xy 133.35 110.49) (xy 133.35 105.41)
-		)
-		(stroke
-			(width 0)
-			(type default)
-		)
-	)
-	(wire
-		(pts
-			(xy 133.35 105.41) (xy 138.43 105.41)
+			(xy 128.27 105.41) (xy 138.43 105.41)
 		)
 		(stroke
@@
 	(wire
 		(pts
-			(xy 128.27 105.41) (xy 133.35 105.41)
-		)
-		(stroke
-			(width 0)
-			(type default)
-		)
-	)
-	(wire
-		(pts
 			(xy 114.3 85.09) (xy 114.3 87.63)
 		)
@@
 		)
 	)
-	(hierarchical_label "MOTOR_IN_2"
+	(wire
+		(pts
+			(xy 128.27 107.95) (xy 138.43 107.95)
+		)
+		(stroke
+			(width 0)
+			(type default)
+		)
+	)
+	(wire
+		(pts
+			(xy 128.27 113.03) (xy 138.43 113.03)
+		)
+		(stroke
+			(width 0)
+			(type default)
+		)
+	)
+	(hierarchical_label "BIN_1_PWM"
 		(shape input)
-		(at 128.27 113.03 180)
+		(at 128.27 110.49 180)
 		(effects
 			(font
@@
 		)
 	)
-	(hierarchical_label "MOTOR_IN_1"
+	(hierarchical_label "AN_1_PWM"
 		(shape input)
 		(at 128.27 105.41 180)
@@
 		)
 	)
-	(hierarchical_label "MOTOR_OUT_2"
-		(shape output)
-		(at 180.34 113.03 0)
+	(hierarchical_label "BIN_2_DIR"
+		(shape input)
+		(at 128.27 113.03 180)
 		(effects
 			(font
 				(size 1.27 1.27)
 			)
-			(justify left)
-		)
-	)
-	(hierarchical_label "MOTOR_OUT_1"
-		(shape output)
-		(at 180.34 105.41 0)
+			(justify right)
+		)
+	)
+	(hierarchical_label "AN_2_DIR"
+		(shape input)
+		(at 128.27 107.95 180)
 		(effects
 			(font
 				(size 1.27 1.27)
 			)
-			(justify left)
+			(justify right)
 		)
 	)
@@
 		(on_board yes)
 		(dnp no)
-		(property "Reference" "#FLG01"
+		(property "Reference" "#FLG02"
 			(at 156.21 78.105 0)
 			(effects
@@
 			(project "esp32-client"
 				(path "/4a001952-2620-48e5-963e-8cfcd99c6e64/53c57007-9e2c-4812-92db-21a9e5c7f42c"
-					(reference "#FLG01")
+					(reference "#FLG02")
 					(unit 1)
 				)
@@
 		(on_board yes)
 		(dnp no)
-		(property "Reference" "#PWR06"
+		(property "Reference" "#PWR07"
 			(at 134.62 82.55 0)
 			(effects
@@
 			(project "esp32-client"
 				(path "/4a001952-2620-48e5-963e-8cfcd99c6e64/53c57007-9e2c-4812-92db-21a9e5c7f42c"
-					(reference "#PWR06")
+					(reference "#PWR07")
 					(unit 1)
 				)
@@
 		(dnp no)
 		(fields_autoplaced yes)
-		(property "Reference" "#PWR04"
+		(property "Reference" "#PWR05"
 			(at 104.14 124.46 0)
 			(effects
@@
 			(project "esp32-client"
 				(path "/4a001952-2620-48e5-963e-8cfcd99c6e64/53c57007-9e2c-4812-92db-21a9e5c7f42c"
-					(reference "#PWR04")
+					(reference "#PWR05")
 					(unit 1)
 				)
@@
 	)
 	(symbol
+		(lib_id "Connector:Conn_01x01_Pin")
+		(at 185.42 105.41 180)
+		(unit 1)
+		(exclude_from_sim no)
+		(in_bom yes)
+		(on_board yes)
+		(dnp no)
+		(fields_autoplaced yes)
+		(property "Reference" "J1"
+			(at 184.785 100.33 0)
+			(effects
+				(font
+					(size 1.27 1.27)
+				)
+			)
+		)
+		(property "Value" "Conn_01x01_Pin"
+			(at 184.785 102.87 0)
+			(effects
+				(font
+					(size 1.27 1.27)
+				)
+			)
+		)
+		(property "Footprint" "Connector_Pin:Pin_D1.0mm_L10.0mm"
+			(at 185.42 105.41 0)
+			(effects
+				(font
+					(size 1.27 1.27)
+				)
+				(hide yes)
+			)
+		)
+		(property "Datasheet" "~"
+			(at 185.42 105.41 0)
+			(effects
+				(font
+					(size 1.27 1.27)
+				)
+				(hide yes)
+			)
+		)
+		(property "Description" "Generic connector, single row, 01x01, script generated"
+			(at 185.42 105.41 0)
+			(effects
+				(font
+					(size 1.27 1.27)
+				)
+				(hide yes)
+			)
+		)
+		(pin "1"
+		)
+		(instances
+			(project ""
+				(path "/4a001952-2620-48e5-963e-8cfcd99c6e64/53c57007-9e2c-4812-92db-21a9e5c7f42c"
+					(reference "J1")
+					(unit 1)
+				)
+			)
+		)
+	)
+	(symbol
 		(lib_id "power:GND")
 		(at 151.13 120.65 0)
@@
 		(dnp no)
 		(fields_autoplaced yes)
-		(property "Reference" "#PWR07"
+		(property "Reference" "#PWR08"
 			(at 151.13 127 0)
 			(effects
@@
 			(project "esp32-client"
 				(path "/4a001952-2620-48e5-963e-8cfcd99c6e64/53c57007-9e2c-4812-92db-21a9e5c7f42c"
-					(reference "#PWR07")
+					(reference "#PWR08")
 					(unit 1)
 				)
@@
 		(dnp no)
 		(fields_autoplaced yes)
-		(property "Reference" "#PWR08"
+		(property "Reference" "#PWR09"
 			(at 158.75 71.12 0)
 			(effects
@@
 			(project ""
 				(path "/4a001952-2620-48e5-963e-8cfcd99c6e64/53c57007-9e2c-4812-92db-21a9e5c7f42c"
-					(reference "#PWR08")
+					(reference "#PWR09")
 					(unit 1)
 				)
@@
 				(path "/4a001952-2620-48e5-963e-8cfcd99c6e64/53c57007-9e2c-4812-92db-21a9e5c7f42c"
 					(reference "C2")
+					(unit 1)
+				)
+			)
+		)
+	)
+	(symbol
+		(lib_id "Connector:Conn_01x01_Pin")
+		(at 185.42 113.03 180)
+		(unit 1)
+		(exclude_from_sim no)
+		(in_bom yes)
+		(on_board yes)
+		(dnp no)
+		(fields_autoplaced yes)
+		(property "Reference" "J2"
+			(at 184.785 107.95 0)
+			(effects
+				(font
+					(size 1.27 1.27)
+				)
+			)
+		)
+		(property "Value" "Conn_01x01_Pin"
+			(at 184.785 110.49 0)
+			(effects
+				(font
+					(size 1.27 1.27)
+				)
+			)
+		)
+		(property "Footprint" "Connector_Pin:Pin_D1.0mm_L10.0mm"
+			(at 185.42 113.03 0)
+			(effects
+				(font
+					(size 1.27 1.27)
+				)
+				(hide yes)
+			)
+		)
+		(property "Datasheet" "~"
+			(at 185.42 113.03 0)
+			(effects
+				(font
+					(size 1.27 1.27)
+				)
+				(hide yes)
+			)
+		)
+		(property "Description" "Generic connector, single row, 01x01, script generated"
+			(at 185.42 113.03 0)
+			(effects
+				(font
+					(size 1.27 1.27)
+				)
+				(hide yes)
+			)
+		)
+		(pin "1"
+		)
+		(instances
+			(project "esp32-client"
+				(path "/4a001952-2620-48e5-963e-8cfcd99c6e64/53c57007-9e2c-4812-92db-21a9e5c7f42c"
+					(reference "J2")
 					(unit 1)
 				)
@@
 		(dnp no)
 		(fields_autoplaced yes)
-		(property "Reference" "#PWR05"
+		(property "Reference" "#PWR06"
 			(at 114.3 93.98 0)
 			(effects
@@
 			(project "esp32-client"
 				(path "/4a001952-2620-48e5-963e-8cfcd99c6e64/53c57007-9e2c-4812-92db-21a9e5c7f42c"
-					(reference "#PWR05")
+					(reference "#PWR06")
 					(unit 1)
 				)

Commit message: init
Parts:
- removed J1, J2: Conn_01x01_Pin, Connector_Pin:Pin_D1.0mm_L10.0mm, symbol Connector:Conn_01x01_Pin
- added J1, J2: Conn_01x02, Connector_JST:JST_EH_B2B-EH-A_1x02_P2.50mm_Vertical, symbol Connector_Generic:Conn_01x02
- R2: footprint Resistor_SMD:R_0805_2012Metric -> Resistor_SMD:R_1206_3216Metric
Connections:
- net at U2.7 (BOUT1): now also J2.1 (Pin_1); no longer U2.2 (AOUT1)
- net at U2.5 (BOUT2): now also J2.2 (Pin_2); no longer U2.4 (AOUT2)
- new net: J1.1 (Pin_1), U2.2 (AOUT1)
- new net: J1.2 (Pin_2), U2.4 (AOUT2)
Changed lines of the file:
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@@
-	)
-	(junction
-		(at 168.91 113.03)
-		(diameter 0)
-		(color 0 0 0 0)
-	)
-	(junction
-		(at 173.99 105.41)
-		(diameter 0)
-		(color 0 0 0 0)
 	)
 	(junction
@@
 	(wire
 		(pts
+			(xy 170.18 113.03) (xy 170.18 120.65)
+		)
+		(stroke
+			(width 0)
+			(type default)
+		)
+	)
+	(wire
+		(pts
 			(xy 156.21 87.63) (xy 156.21 82.55)
 		)
@@
 	(wire
 		(pts
-			(xy 173.99 110.49) (xy 173.99 105.41)
-		)
-		(stroke
-			(width 0)
-			(type default)
-		)
-	)
-	(wire
-		(pts
 			(xy 140.97 82.55) (xy 144.78 82.55)
 		)
@@
 	(wire
 		(pts
-			(xy 163.83 110.49) (xy 173.99 110.49)
+			(xy 163.83 107.95) (xy 180.34 107.95)
 		)
 		(stroke
@@
 	(wire
 		(pts
-			(xy 168.91 113.03) (xy 180.34 113.03)
+			(xy 170.18 120.65) (xy 180.34 120.65)
 		)
 		(stroke
@@
 	(wire
 		(pts
-			(xy 163.83 113.03) (xy 168.91 113.03)
-		)
-		(stroke
-			(width 0)
-			(type default)
-		)
-	)
-	(wire
-		(pts
-			(xy 163.83 107.95) (xy 168.91 107.95)
-		)
-		(stroke
-			(width 0)
-			(type default)
-		)
-	)
-	(wire
-		(pts
-			(xy 168.91 107.95) (xy 168.91 113.03)
+			(xy 163.83 110.49) (xy 175.26 110.49)
 		)
 		(stroke
@@
 	(wire
 		(pts
-			(xy 163.83 105.41) (xy 173.99 105.41)
-		)
-		(stroke
-			(width 0)
-			(type default)
-		)
-	)
-	(wire
-		(pts
 			(xy 128.27 105.41) (xy 138.43 105.41)
 		)
@@
 	(wire
 		(pts
+			(xy 163.83 105.41) (xy 180.34 105.41)
+		)
+		(stroke
+			(width 0)
+			(type default)
+		)
+	)
+	(wire
+		(pts
 			(xy 151.13 118.11) (xy 151.13 120.65)
 		)
@@
 	(wire
 		(pts
-			(xy 173.99 105.41) (xy 180.34 105.41)
+			(xy 163.83 113.03) (xy 170.18 113.03)
 		)
 		(stroke
@@
 		(pts
 			(xy 114.3 85.09) (xy 114.3 87.63)
+		)
+		(stroke
+			(width 0)
+			(type default)
+		)
+	)
+	(wire
+		(pts
+			(xy 175.26 118.11) (xy 180.34 118.11)
+		)
+		(stroke
+			(width 0)
+			(type default)
+		)
+	)
+	(wire
+		(pts
+			(xy 175.26 110.49) (xy 175.26 118.11)
 		)
 		(stroke
@@
 			)
 		)
-		(property "Footprint" "Resistor_SMD:R_0805_2012Metric"
+		(property "Footprint" "Resistor_SMD:R_1206_3216Metric"
 			(at 102.362 110.49 90)
 			(effects
@@
 	)
 	(symbol
-		(lib_id "Connector:Conn_01x01_Pin")
-		(at 185.42 105.41 180)
+		(lib_id "Connector_Generic:Conn_01x02")
+		(at 185.42 118.11 0)
 		(unit 1)
 		(exclude_from_sim no)
@@
 		(dnp no)
 		(fields_autoplaced yes)
-		(property "Reference" "J1"
-			(at 184.785 100.33 0)
-			(effects
-				(font
-					(size 1.27 1.27)
-				)
-			)
-		)
-		(property "Value" "Conn_01x01_Pin"
-			(at 184.785 102.87 0)
-			(effects
-				(font
-					(size 1.27 1.27)
-				)
-			)
-		)
-		(property "Footprint" "Connector_Pin:Pin_D1.0mm_L10.0mm"
-			(at 185.42 105.41 0)
+		(property "Reference" "J2"
+			(at 187.96 118.1099 0)
+			(effects
+				(font
+					(size 1.27 1.27)
+				)
+				(justify left)
+			)
+		)
+		(property "Value" "Conn_01x02"
+			(at 187.96 120.6499 0)
+			(effects
+				(font
+					(size 1.27 1.27)
+				)
+				(justify left)
+			)
+		)
+		(property "Footprint" "Connector_JST:JST_EH_B2B-EH-A_1x02_P2.50mm_Vertical"
+			(at 185.42 118.11 0)
 			(effects
 				(font
@@
 		)
 		(property "Datasheet" "~"
-			(at 185.42 105.41 0)
-			(effects
-				(font
-					(size 1.27 1.27)
-				)
-				(hide yes)
-			)
-		)
-		(property "Description" "Generic connector, single row, 01x01, script generated"
-			(at 185.42 105.41 0)
+			(at 185.42 118.11 0)
+			(effects
+				(font
+					(size 1.27 1.27)
+				)
+				(hide yes)
+			)
+		)
+		(property "Description" "Generic connector, single row, 01x02, script generated (kicad-library-utils/schlib/autogen/connector/)"
+			(at 185.42 118.11 0)
 			(effects
 				(font
@@
 		)
 		(pin "1"
+		)
+		(pin "2"
 		)
 		(instances
 			(project ""
 				(path "/4a001952-2620-48e5-963e-8cfcd99c6e64/53c57007-9e2c-4812-92db-21a9e5c7f42c"
-					(reference "J1")
+					(reference "J2")
 					(unit 1)
 				)
@@
 	)
 	(symbol
-		(lib_id "Connector:Conn_01x01_Pin")
-		(at 185.42 113.03 180)
-		(unit 1)
-		(exclude_from_sim no)
-		(in_bom yes)
-		(on_board yes)
-		(dnp no)
-		(fields_autoplaced yes)
-		(property "Reference" "J2"
-			(at 184.785 107.95 0)
-			(effects
-				(font
-					(size 1.27 1.27)
-				)
-			)
-		)
-		(property "Value" "Conn_01x01_Pin"
-			(at 184.785 110.49 0)
-			(effects
-				(font
-					(size 1.27 1.27)
-				)
-			)
-		)
-		(property "Footprint" "Connector_Pin:Pin_D1.0mm_L10.0mm"
-			(at 185.42 113.03 0)
-			(effects
-				(font
-					(size 1.27 1.27)
-				)
-				(hide yes)
-			)
-		)
-		(property "Datasheet" "~"
-			(at 185.42 113.03 0)
-			(effects
-				(font
-					(size 1.27 1.27)
-				)
-				(hide yes)
-			)
-		)
-		(property "Description" "Generic connector, single row, 01x01, script generated"
-			(at 185.42 113.03 0)
-			(effects
-				(font
-					(size 1.27 1.27)
-				)
-				(hide yes)
-			)
-		)
-		(pin "1"
-		)
-		(instances
-			(project "esp32-client"
-				(path "/4a001952-2620-48e5-963e-8cfcd99c6e64/53c57007-9e2c-4812-92db-21a9e5c7f42c"
-					(reference "J2")
-					(unit 1)
-				)
-			)
-		)
-	)
-	(symbol
 		(lib_id "Driver_Motor:DRV8833PW")
 		(at 151.13 102.87 0)
@@
 					(unit 1)
 				)
+			)
+		)
+	)
+	(symbol
+		(lib_id "Connector_Generic:Conn_01x02")
+		(at 185.42 105.41 0)
+		(unit 1)
+		(exclude_from_sim no)
+		(in_bom yes)
+		(on_board yes)
+		(dnp no)
+		(fields_autoplaced yes)
+		(property "Reference" "J1"
+			(at 187.96 105.4099 0)
+			(effects
+				(font
+					(size 1.27 1.27)
+				)
+				(justify left)
+			)
+		)
+		(property "Value" "Conn_01x02"
+			(at 187.96 107.9499 0)
+			(effects
+				(font
+					(size 1.27 1.27)
+				)
+				(justify left)
+			)
+		)
+		(property "Footprint" "Connector_JST:JST_EH_B2B-EH-A_1x02_P2.50mm_Vertical"
+			(at 185.42 105.41 0)
+			(effects
+				(font
+					(size 1.27 1.27)
+				)
+				(hide yes)
+			)
+		)
+		(property "Datasheet" "~"
+			(at 185.42 105.41 0)
+			(effects
+				(font
+					(size 1.27 1.27)
+				)
+				(hide yes)
+			)
+		)
+		(property "Description" "Generic connector, single row, 01x02, script generated (kicad-library-utils/schlib/autogen/connector/)"
+			(at 185.42 105.41 0)
+			(effects
+				(font
+					(size 1.27 1.27)
+				)
+				(hide yes)
+			)
+		)
+		(pin "2"
+		)
+		(pin "1"
+		)
+		(instances
+			(project ""
+				(path "/4a001952-2620-48e5-963e-8cfcd99c6e64/53c57007-9e2c-4812-92db-21a9e5c7f42c"
+					(reference "J1")
+					(unit 1)
+				)
