File: kicad/esp32-client.kicad_pcb (KiCad board)
At the start: 2 copper layers, 36 x 56 mm, 42 parts, among them J1 Conn_01x01_Pin, J2 Conn_01x01_Pin, J3 Conn_01x02, P1 USB_C_Plug_USB2.0, Q1 BCW66G, Q2 BCW66G, U1 ESP32-C3-MINI-1, U2 DRV8833PW, U3 TP4056-42-ESOP8, U4 U8205A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

Commit message: init
Parts:
- J1, J2: value Conn_01x01_Pin -> Conn_01x02; footprint Connector_Pin:Pin_D1.0mm_L10.0mm -> Connector_JST:JST_EH_B2B-EH-A_1x02_P2.50mm_Vertical
- R1, R10, R11, R12, R2, R3, R4, R5, R6, R7, R8, R9: footprint Resistor_SMD:R_0805_2012Metric -> Resistor_SMD:R_1206_3216Metric
- moved D2 13.3 mm to (197.0, 67.5), turned to 180 degrees
- moved J1 9.25 mm to (203.2, 71.8)
- moved J3 8.54 mm to (192.0, 72.0)
- moved U5 7.52 mm to (175.0, 83.0)
- moved C1 6.53 mm to (174.0, 74.0)
- moved C3 5.83 mm to (190.5, 78.5)
- moved U4 4.64 mm to (181.0, 83.0)
- moved J2 4.03 mm to (203.0, 61.0), turned to 90 degrees
- moved C2 3.81 mm to (183.5, 75.5)
- moved R8 3.56 mm to (179.5, 75.0)
- moved R6 3.54 mm to (180.0, 70.0)
- moved C4 3.35 mm to (186.5, 82.5), turned to 90 degrees
- moved R2 2.90 mm to (200.0, 77.0), turned to 0 degrees
- moved C6 2.00 mm to (194.5, 78.5), turned to 90 degrees
- moved C8 1.80 mm to (174.0, 70.0)
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Connections:
- U2 pad 4: Net-(J2-Pin_1) -> Net-(J1-Pin_2)
- U2 pad 5: Net-(J2-Pin_1) -> Net-(J2-Pin_2)
- U2 pad 7: Net-(J1-Pin_1) -> Net-(J2-Pin_1)
Routing:
- net GND: track 278.4 -> 0.00 mm, vias 4 -> 0
- net +5V: track 138.9 -> 0.00 mm, vias 2 -> 0
- net +3.3V: track 119.7 -> 0.00 mm, vias 5 -> 0
- net /power/EN: track 86.6 -> 0.00 mm, vias 2 -> 0
- net Net-(Q2-E): track 61.3 -> 0.00 mm, vias 4 -> 0
- net /power/TXD: track 57.5 -> 0.00 mm, vias 2 -> 0
- net /power/RXD: track 55.1 -> 0.00 mm, vias 4 -> 0
- net Net-(Q1-E): track 54.3 -> 0.00 mm, vias 4 -> 0
- net Net-(U3-TEMP): track 38.9 -> 0.00 mm, vias 3 -> 0
- net Net-(U2-VINT): track 37.3 -> 0.00 mm, vias 2 -> 0
- net Net-(J3-Pin_1): track 31.4 -> 0.00 mm, vias 3 -> 0
- net Net-(U7-UD+): track 29.7 -> 0.00 mm, vias 2 -> 0
- net /motor_driver/AN_1_PWM: track 27.7 -> 0.00 mm, vias 2 -> 0
- net Net-(U2-AISEN): track 27.6 -> 0.00 mm
- net /motor_driver/AN_2_DIR: track 27.2 -> 0.00 mm, vias 2 -> 0
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
Commit message: init
Parts:
- removed C9: 100nF, Capacitor_SMD:C_1206_3216Metric
- removed Q1, Q2: BCW66G, Package_TO_SOT_SMD:SOT-23
- removed R10, R11: 10K, Resistor_SMD:R_1206_3216Metric
- removed U7: CH340C, Package_SO:SOIC-16_3.9x9.9mm_P1.27mm
- moved U5 16.2 mm to (177.5, 99.0)
- moved R8 10.6 mm to (178.0, 85.5)
- moved U4 10.1 mm to (177.5, 92.5)
- moved C2 4.61 mm to (180.5, 79.0)
Connections:
- net /power/EN renamed Net-(U1-EN/CHIP_PU)
- C6 pad 1: Net-(J3-Pin_1) -> +3.3V
- C7 pad 1: Net-(U5-GND) -> Net-(J3-Pin_2)
- J3 pad 1: Net-(J3-Pin_1) -> +3.3V
- J3 pad 2: GND -> Net-(J3-Pin_2)
- R9 pad 1: Net-(U5-VCC) -> +3.3V
- R9 pad 2: Net-(J3-Pin_1) -> Net-(U5-VCC)
- U1 pad 12: /power/IO0 -> unconnected-(U1-GPIO0/ADC1_CH0/XTAL_32K_P-Pad12)
- U1 pad 26: unconnected-(U1-GPIO18/USB_D--Pad26) -> /power/D-
- U1 pad 27: unconnected-(U1-GPIO19/USB_D+-Pad27) -> /power/D+
- U1 pad 30: /power/TXD -> unconnected-(U1-GPIO20/U0RXD-Pad30)
- U1 pad 31: /power/RXD -> unconnected-(U1-GPIO21/U0TXD-Pad31)
- U3 pad 5: Net-(J3-Pin_1) -> +3.3V
- U4 pad 3: GND -> Net-(J3-Pin_2)
- U5 pad 6: Net-(U5-GND) -> Net-(J3-Pin_2)
- U6 pad 4: Net-(U7-UD-) -> /power/D-
- U6 pad 6: Net-(U7-UD+) -> /power/D+

Commit message: init
Parts:
- C2: footprint Capacitor_THT:CP_Radial_D5.0mm_P2.00mm -> Capacitor_SMD:CP_Elec_6.3x4.5
- moved C4 6.95 mm to (180.5, 86.0)
- moved R8 5.00 mm to (174.0, 82.5), turned to 180 degrees
- moved R12 4.77 mm to (181.5, 99.0)
- moved R7 3.60 mm to (187.0, 98.5), turned to 0 degrees
- moved U5 3.04 mm to (174.5, 99.5)
- moved C2 2.83 mm to (182.5, 77.0), turned to 90 degrees
- moved U2 2.06 mm to (194.5, 60.0)
- moved C10 1.79 mm to (174.0, 87.0), turned to 0 degrees
- moved R9 1.59 mm to (190.0, 93.0)
- moved U4 1.00 mm to (178.4, 92.0)
- moved J2 0.20 mm to (203.2, 61.0)

Commit message: init
Parts:
- moved C10 2.00 mm to (174.0, 89.0)
- moved R8 1.50 mm to (174.0, 84.0)
- moved U4 1.50 mm to (178.4, 93.5)
- moved C5 1.00 mm to (174.0, 79.0)
- moved C1 0.50 mm to (174.0, 74.5)
Changed lines of the file:
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@@
 	(footprint "Package_TO_SOT_SMD:SOT-23-6"
 		(layer "F.Cu")
-		(at 178.3625 92)
+		(at 178.3625 93.5)
 		(descr "SOT, 6 Pin (JEDEC MO-178 Var AB https://www.jedec.org/document_search?search_api_views_fulltext=MO-178), generated with kicad-footprint-generator ipc_gullwing_generator.py")
 		(tags "SOT TO_SOT_SMD")
@@
 	(footprint "Capacitor_SMD:C_1206_3216Metric"
 		(layer "F.Cu")
-		(at 174 78)
+		(at 174 79)
 		(descr "Capacitor SMD 1206 (3216 Metric), square (rectangular) end terminal, IPC-7351 nominal, (Body size source: IPC-SM-782 page 76, https://www.pcb-3d.com/wordpress/wp-content/uploads/ipc-sm-782a_amendment_1_and_2.pdf), generated with kicad-footprint-generator")
 		(tags "capacitor")
@@
 	(footprint "Capacitor_SMD:C_1206_3216Metric"
 		(layer "F.Cu")
-		(at 174 87)
+		(at 174 89)
 		(descr "Capacitor SMD 1206 (3216 Metric), square (rectangular) end terminal, IPC-7351 nominal, (Body size source: IPC-SM-782 page 76, https://www.pcb-3d.com/wordpress/wp-content/uploads/ipc-sm-782a_amendment_1_and_2.pdf), generated with kicad-footprint-generator")
 		(tags "capacitor")
 		(property "Reference" "C10"
-			(at 3.975 -1 0)
+			(at 0 -2.5 0)
 			(layer "F.SilkS")
 			(effects
@@
 	(footprint "Resistor_SMD:R_1206_3216Metric"
 		(layer "F.Cu")
-		(at 174 82.5 180)
+		(at 174 84 180)
 		(descr "Resistor SMD 1206 (3216 Metric), square (rectangular) end terminal, IPC-7351 nominal, (Body size source: IPC-SM-782 page 72, https://www.pcb-3d.com/wordpress/wp-content/uploads/ipc-sm-782a_amendment_1_and_2.pdf), generated with kicad-footprint-generator")
 		(tags "resistor")
@@
 	(footprint "Capacitor_SMD:C_1206_3216Metric"
 		(layer "F.Cu")
-		(at 174 74)
+		(at 174 74.5)
 		(descr "Capacitor SMD 1206 (3216 Metric), square (rectangular) end terminal, IPC-7351 nominal, (Body size source: IPC-SM-782 page 76, https://www.pcb-3d.com/wordpress/wp-content/uploads/ipc-sm-782a_amendment_1_and_2.pdf), generated with kicad-footprint-generator")
 		(tags "capacitor")

Commit message: init
Routing:
- net +3.3V: track 0.00 -> 149.2 mm, vias 0 -> 6
- net +5V: track 0.00 -> 134.5 mm, vias 0 -> 3
- net Net-(U1-EN/CHIP_PU): track 0.00 -> 59.3 mm
- net /power/D+: track 0.00 -> 54.3 mm, vias 0 -> 2
- net Net-(J3-Pin_2): track 0.00 -> 51.6 mm, vias 0 -> 2
- net Net-(U3-TEMP): track 0.00 -> 40.3 mm
- net /power/D-: track 0.00 -> 38.5 mm, vias 0 -> 2
- net Net-(U2-VINT): track 0.00 -> 36.5 mm, vias 0 -> 2
- net Net-(U2-AISEN): track 0.00 -> 25.0 mm
- net /motor_driver/SLEEP: track 0.00 -> 24.8 mm, vias 0 -> 2
- net /motor_driver/AN_2_DIR: track 0.00 -> 24.7 mm, vias 0 -> 2
- net Net-(U2-VCP): track 0.00 -> 24.1 mm
- net /motor_driver/AN_1_PWM: track 0.00 -> 23.8 mm, vias 0 -> 2
- net Net-(U5-VCC): track 0.00 -> 22.6 mm, vias 0 -> 2
- net Net-(U3-PROG): track 0.00 -> 22.3 mm, vias 0 -> 2
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
Commit message: init
Parts:
- moved C7 2.55 mm to (185.0, 86.0), turned to -90 degrees
- moved D2 1.71 mm to (197.0, 65.8), turned to 90 degrees
- moved R5 1.62 mm to (191.5, 66.0), turned to 90 degrees
- moved U3 1.41 mm to (191.8, 86.2)
- moved R4 1.00 mm to (204.0, 87.5)
- moved U2 1.00 mm to (194.5, 59.0), turned to 180 degrees
- turned R2 to 180 degrees
- turned U4 to -90 degrees
Routing:
- net GND: track 0.70 -> 201.5 mm, vias 0 -> 21
- net +3.3V: track 149.2 -> 133.8 mm
- net /motor_driver/AN_2_DIR: track 24.7 -> 17.6 mm
- net Net-(J1-Pin_1): track 20.0 -> 14.0 mm
- net Net-(J2-Pin_2): track 11.5 -> 5.91 mm, vias 1 -> 0
- net Net-(U2-VINT): track 36.5 -> 30.9 mm, vias 2 -> 0
- net Net-(D2-K): track 22.1 -> 26.8 mm, vias 0 -> 2
- net +5V: track 134.5 -> 130.0 mm, vias 3 -> 2
- net /motor_driver/AN_1_PWM: track 23.8 -> 19.5 mm
- net Net-(U3-~{STDBY}): track 10.3 -> 14.2 mm, vias 0 -> 2
- net Net-(U4-G2): track 15.7 -> 12.1 mm
- net Net-(J1-Pin_2): track 15.6 -> 12.7 mm, vias 1 -> 0
- net /power/D+: track 54.3 -> 51.8 mm
- net /motor_driver/BIN_1_PWM: track 17.7 -> 20.1 mm
- net Net-(U5-VCC): track 22.6 -> 24.8 mm
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
Commit message: init
Parts:
- removed C11: 10µF, Capacitor_SMD:C_1206_3216Metric
- removed R12: 2K, Resistor_SMD:R_1206_3216Metric
- added C9: 10µF, Capacitor_SMD:C_1206_3216Metric, F.Cu at (216.6, 72.7)
- added R10: 100, Resistor_SMD:R_1206_3216Metric, F.Cu at (216.5, 76.0)
- added U7: ~, PCM_yvolodym:Switch, F.Cu at (215.5, 91.0)
- C10: value 10µF -> 100nF
- C8: value 100nF -> 10µF
- R9: value 100 -> 2K
- U4: value U8205A -> USBLC6-2P6
- U5: value DW01A -> U8205A
- U6: value USBLC6-2P6 -> DW01A
Connections:
- C10 pad 1: +5V -> GND
- C10 pad 2: GND -> +5V
- C7 pad 1: Net-(J3-Pin_2) -> Net-(U5-S2)
- C7 pad 2: Net-(U5-VCC) -> Net-(U6-VCC)
- C8 pad 1: GND -> +5V
- C8 pad 2: +5V -> GND
- R8 pad 2: Net-(U5-CS) -> Net-(U6-CS)
- R9 pad 1: +3.3V -> +5V
- R9 pad 2: Net-(U5-VCC) -> Net-(D3-A)
- U4 pad 1: GND -> Net-(P1-D+)
- U4 pad 2: unconnected-(U4-D1-Pad2) -> GND
- U4 pad 3: Net-(J3-Pin_2) -> Net-(P1-D-)
- U4 pad 4: Net-(U4-G2) -> /power/D-
- U4 pad 5: unconnected-(U4-D2-Pad5) -> +5V
- U4 pad 6: Net-(U4-G1) -> /power/D+
- U5 pad 1: Net-(U4-G2) -> GND
- U5 pad 2: Net-(U5-CS) -> unconnected-(U5-D1-Pad2)
- U5 pad 3: Net-(U4-G1) -> Net-(U5-S2)
- U5 pad 4: unconnected-(U5-TD-Pad4) -> Net-(U5-G2)
- U5 pad 5: Net-(U5-VCC) -> unconnected-(U5-D2-Pad5)
- U5 pad 6: Net-(J3-Pin_2) -> Net-(U5-G1)
- U6 pad 1: Net-(P1-D+) -> Net-(U5-G2)
- U6 pad 2: GND -> Net-(U6-CS)
- U6 pad 3: Net-(P1-D-) -> Net-(U5-G1)
- U6 pad 4: /power/D- -> unconnected-(U6-TD-Pad4)
- U6 pad 5: +5V -> Net-(U6-VCC)
- U6 pad 6: /power/D+ -> Net-(U5-S2)
Routing:
- net (no net): track 0.00 -> 29.1 mm
- net Net-(U5-VCC): track 24.8 -> 0.00 mm, vias 2 -> 0
- net Net-(D3-A): track 5.49 -> 30.3 mm, vias 0 -> 2
- net Net-(U5-CS): track 17.0 -> 0.00 mm
- net Net-(U4-G2): track 12.1 -> 0.00 mm
- net Net-(U4-G1): track 11.7 -> 0.00 mm
- net /power/D+: track 51.8 -> 63.5 mm

Commit message: init
Parts:
- C2: footprint Capacitor_SMD:CP_Elec_6.3x4.5 -> Capacitor_SMD:CP_Elec_4x3.9
