File: kicad/esp32-client.kicad_pcb (KiCad board)
At the start: 2 copper layers, 36 x 56 mm, 37 parts, among them J1 Conn_01x02, J2 Conn_01x02, J3 Conn_01x02, P1 USB_C_Plug_USB2.0, U1 ESP32-C3-MINI-1, U2 DRV8833PW, U3 TP4056-42-ESOP8, U4 USBLC6-2P6, U5 U8205A, U6 DW01A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

Commit message: init
Parts:
- moved R1 49.0 mm to (174.0, 58.5)
- moved C9 48.7 mm to (181.0, 106.0), turned to -90 degrees
- moved R10 43.2 mm to (173.5, 72.0), turned to 90 degrees
- moved U7 34.7 mm to (181.0, 94.5), turned to 180 degrees
- moved J3 32.8 mm to (173.5, 99.0), turned to 90 degrees
- moved R4 30.7 mm to (177.5, 72.0)
- moved C8 30.6 mm to (187.5, 97.5), turned to -90 degrees
- moved D2 29.7 mm to (173.0, 83.3)
- moved C4 26.2 mm to (195.5, 64.5), turned to 180 degrees
- moved U6 24.4 mm to (176.5, 78.6), turned to -90 degrees
- moved R3 23.9 mm to (182.5, 80.5), turned to 90 degrees
- moved D1 23.6 mm to (174.8, 92.5), turned to 0 degrees
- moved H1 23.6 mm to (202.5, 59.0)
- moved C2 21.4 mm to (203.0, 70.8)
- moved C5 20.9 mm to (194.5, 83.0)
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Routing:
- net Net-(U1-EN/CHIP_PU): track 59.2 -> 7.22 mm
- net Net-(J3-Pin_2): track 50.4 -> 8.54 mm, vias 1 -> 0
- net Net-(U5-S2): track 0.00 -> 32.3 mm
- net Net-(U6-CS): track 0.00 -> 31.1 mm, vias 0 -> 2
- net (no net): track 29.1 -> 0.00 mm
- net +5V: track 130.0 -> 101.5 mm
- net Net-(U3-~{CHRG}): track 11.1 -> 38.9 mm
- net Net-(D3-A): track 30.3 -> 5.14 mm, vias 2 -> 0
- net GND: track 201.5 -> 221.4 mm, vias 21 -> 2
- net Net-(U6-VCC): track 0.00 -> 19.4 mm
- net Net-(U5-G2): track 0.00 -> 19.0 mm, vias 0 -> 2
- net Net-(U2-VINT): track 30.9 -> 12.0 mm
- net +3.3V: track 133.8 -> 151.7 mm, vias 6 -> 3
- net Net-(U3-TEMP): track 40.0 -> 24.4 mm, vias 3 -> 2
- net Net-(U3-PROG): track 23.8 -> 8.32 mm
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